File: KiCAD/PV16SOG.sch (KiCad schematic (older format))
At the start: 57 parts, among them CON1 BARREL_JACK 2,1mm, J1 RCA_JACK, J2 RCA_JACK, J3 DB9, J4 PS/2, P1 ICSP, SW1 Power, SW2 reset, U1 LD33V, U2 PIC24EP512MC202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

Commit message: ajout schematic.pdf
Parts:
- C9: symbol CP -> CP-RESCUE-PV16SOG
- RV1: symbol POT -> POT-RESCUE-PV16SOG
Connections:
- net at R11.2: now also RV1.1
Changed lines of the file:
@@
 $EndComp
 $Comp
-L POT RV1
+L POT-RESCUE-PV16SOG RV1
 U 1 1 56343FFC
 P 4150 5750
@@
 2
 $Comp
-L CP C9
+L CP-RESCUE-PV16SOG C9
 U 1 1 5684AC91
 P 6500 4800
@@
 	1550 600  2250 600
 Wire Wire Line
-	3800 5750 3900 5750
+	3800 5750 4000 5750
 Connection ~ 6200 4800
 Wire Wire Line
